Commit message: MAJ 19 avril 2020

File: urdf/turtlebot3_burger.gazebo.xacro (robot description, xacro)
@@ -3,12 +3,10 @@
   <xacro:arg name="laser_visual" default="false"/>
   <xacro:arg name="imu_visual"   default="false"/>
-  <xacro:property name="yaml_file" value="$(find challenge_project)/config/turtlebot3_burger.yaml" />
-  <xacro:property name="props" value="${load_yaml(yaml_file)}"/>
   <gazebo reference="base_link">
     <material>Gazebo/DarkGrey</material>
   </gazebo>
   <gazebo reference="wheel_left_link">
-    <mu1>0.1</mu1>
-    <mu2>0.1</mu2>
+    <mu1>1</mu1>
+    <mu2>1</mu2>
     <kp>500000.0</kp>
     <kd>10.0</kd>
@@ -19,6 +17,6 @@
   </gazebo>
   <gazebo reference="wheel_right_link">
-    <mu1>0.1</mu1>
-    <mu2>0.1</mu2>
+    <mu1>1</mu1>
+    <mu2>1</mu2>
     <kp>500000.0</kp>
     <kd>10.0</kd>
@@ -44,8 +42,7 @@
     <material>Gazebo/FlatBlack</material>
   </gazebo>
-  <xacro:property name="motorsCommandTopic" value="${props['motorsCommandTopic']}" />
   <gazebo>
     <plugin name="turtlebot3_burger_controller" filename="libgazebo_ros_diff_drive.so">
-      <commandTopic>${motorsCommandTopic}</commandTopic>
+      <commandTopic>cmd_vel</commandTopic>
       <odometryTopic>odom</odometryTopic>
       <odometryFrame>odom</odometryFrame>
@@ -95,11 +92,4 @@
     </plugin>
   </gazebo>
-  <xacro:property name="lds_scan_samples" value="${props['lds_scan_samples']}" />
-  <xacro:property name="lds_scan_resolution" value="${props['lds_scan_resolution']}" />
-  <xacro:property name="lds_scan_angle" value="${props['lds_scan_angle']}" />
-  <xacro:property name="lds_range" value="${props['lds_range']}" />
-  <xacro:property name="lds_range_resolution" value="${props['lds_range_resolution']}" />
-  <xacro:property name="ldsTopicName" value="${props['ldsTopicName']}" />
-  <xacro:property name="ldsFrameName" value="${props['ldsFrameName']}" />
   <gazebo reference="base_scan">
     <material>Gazebo/FlatBlack</material>
@@ -111,14 +101,14 @@
         <scan>
           <horizontal>
-            <samples>${lds_scan_samples}</samples>
-            <resolution>${lds_scan_resolution}</resolution>
-            <min_angle>${lds_scan_angle[0]}</min_angle>
-            <max_angle>${lds_scan_angle[1]}</max_angle>
+            <samples>360</samples>
+            <resolution>1</resolution>
+            <min_angle>0.0</min_angle>
+            <max_angle>6.28319</max_angle>
           </horizontal>
         </scan>
         <range>
-          <min>${lds_range[0]}</min>
-          <max>${lds_range[1]}</max>
-          <resolution>${lds_range_resolution}</resolution>
+          <min>0.120</min>
+          <max>3.5</max>
+          <resolution>0.015</resolution>
         </range>
         <noise>
@@ -129,30 +119,23 @@
       </ray>
       <plugin name="gazebo_ros_lds_lfcd_controller" filename="libgazebo_ros_laser.so">
-        <topicName>${ldsTopicName}</topicName>
-        <frameName>${ldsFrameName}</frameName>
+        <topicName>scan</topicName>
+        <frameName>base_scan</frameName>
       </plugin>
     </sensor>
   </gazebo>
-  <xacro:property name="cam_rate" value="${props['cam_rate']}" />
-  <xacro:property name="cam_fov" value="${props['cam_fov']}" />
-  <xacro:property name="cam_image_size" value="${props['cam_image_size']}" />
-  <xacro:property name="cam_range" value="${props['cam_range']}" />
-  <xacro:property name="motors_rate" value="${props['val1']}" />
-  <xacro:property name="imageTopicName" value="${props['imageTopicName']}" />
-  <xacro:property name="imageInfoTopicName" value="${props['imageInfoTopicName']}" />
  <!-- camera -->
   <gazebo reference="camera_link">
     <sensor type="camera" name="camera1">
-      <update_rate>${cam_rate}</update_rate>
+      <update_rate>30.0</update_rate>
       <camera name="head">
-        <horizontal_fov>${cam_fov}</horizontal_fov>
+        <horizontal_fov>1.3962634</horizontal_fov>
         <image>
-          <width>${cam_image_size[0]}</width>
-          <height>${cam_image_size[1]}</height>
+          <width>800</width>
+          <height>800</height>
           <format>R8G8B8</format>
         </image>
         <clip>
-          <near>${cam_range[0]}</near>
-          <far>${cam_range[1]}</far>
+          <near>0.02</near>
+          <far>300</far>
         </clip>
         <noise>
@@ -169,6 +152,6 @@
         <updateRate>30.0</updateRate> <!--images prises par seconde -->
         <cameraName></cameraName> <!-- nom de la camera -->
-        <imageTopicName>${imageTopicName}</imageTopicName>
-        <cameraInfoTopicName>${imageInfoTopicName}</cameraInfoTopicName>
+        <imageTopicName>camera/image_raw</imageTopicName>
+        <cameraInfoTopicName>camera/camera_info</cameraInfoTopicName>
         <frameName>camera_link</frameName>
         <hackBaseline>0.07</hackBaseline>

File: urdf/turtlebot3_burger.urdf.xacro (robot description, xacro)
@@ -1,11 +1,7 @@
 <?xml version="1.0" ?>
 <robot name="turtlebot3_burger" xmlns:xacro="http://ros.org/wiki/xacro">
-  <xacro:include filename="$(find challenge_project)/urdf/turtlebot3_burger/common_properties.xacro"/>
-  <xacro:include filename="$(find challenge_project)/urdf/turtlebot3_burger/turtlebot3_burger.gazebo.xacro"/>
-  <xacro:property name="yaml_file" value="$(find challenge_project)/config/turtlebot3_burger.yaml" />
-  <xacro:property name="props" value="${load_yaml(yaml_file)}"/>
-  <xacro:property name="camera_link" value="0.015" /> <!-- Size of square 'camera' box -->
-  <xacro:property name="cam_ori" value="${props['cam_orientation']}" />
-  <xacro:property name="cam_pos" value="${props['cam_position']}" />
+  <xacro:include filename="$(find challenge_project)/urdf/common_properties.xacro"/>
+  <xacro:include filename="$(find challenge_project)/urdf/turtlebot3_burger.gazebo.xacro"/>
+    <xacro:property name="camera_link" value="0.015" /> <!-- Size of square 'camera' box -->
   <link name="base_footprint"/>
   <joint name="base_joint" type="fixed">
@@ -168,6 +164,5 @@
  <joint name="camera_joint" type="fixed">
     <axis xyz="0 1 0" />
-    <origin xyz="${cam_pos[0]} ${cam_pos[1]} ${cam_pos[2]}"
-	    rpy="${cam_ori[0]} ${cam_ori[1]} ${cam_ori[2]}"/> <!--position et orientation de la camera-->
+    <origin xyz="0.03 0 0.125" rpy="0 0.610865238 0"/> <!--position et orientation de la camera-->
     <parent link="base_link"/>
     <child link="camera_link"/>
